File: DRV8833Motordriver.kicad_sch (KiCad schematic)
At the start: 0 parts

Commit message: Added all Components to Schematic
Parts:
- added C1, C2, C3: C, symbol Device:C
- added D1: LED, symbol Device:LED
- added J1, J2: Conn_01x06_Pin, symbol Connector:Conn_01x06_Pin
- added R1: R, symbol Device:R
- added U1: DRV8833PWP, Package_SO:HTSSOP-16-1EP_4.4x5mm_P0.65mm_EP3.4x5mm_Mask2.46x2.31mm_ThermalVias, symbol Driver_Motor:DRV8833PWP
Connections:
- new net: U1.13 (GND), U1.17 (GND)
