File: DRV8833Motordriver.kicad_pcb (KiCad board)
At the start: 2 copper layers, 32.2 x 19.8 mm, 8 parts, among them J1 Conn_01x06_Pin, J2 Conn_01x06_Pin, U1 DRV8833PWP

Commit message: PCB with 0 DRC Errors
Routing:
- net /BOUT1: track 17.2 -> 14.8 mm
- net GND: track 50.5 -> 49.3 mm
- net /VCC: track 58.9 -> 59.6 mm
- net Net-(D1-K): track 6.38 -> 6.97 mm
